Commit message: Work on camera plugin

File: tello_description/urdf/tello.urdf (robot description, URDF)
Before this commit: robot tello, 2 links, 1 joints
Links:
- removed link camera_frame
- added link camera_link, mass 1e-5; collision sphere radius=0.01; visual sphere radius=0.01
Joints:
- joint camera_joint: child camera_frame -> camera_link; origin xyz=0.035 0 0 rpy=1.5708 3.1416 1.5708 -> xyz=0.035 0 0 rpy=0 0 0
